Commit message: first commit

File: mycobot_ros/mycobot_description/urdf/280_arduino/mycobot_urdf_fake.urdf (robot description, URDF)
Before this commit: robot firefighter, 8 links, 7 joints
Links:
- removed link apriltag
- link joint1: geometry collision box size=0.01 0.01 0.01; visual box size=0.01 0.01 0.01
- link joint2: geometry collision box size=0.01 0.01 0.01; visual box size=0.01 0.01 0.01
- link joint3: geometry collision box size=0.01 0.01 0.01; visual box size=0.01 0.01 0.01
- link joint4: geometry collision box size=0.01 0.01 0.01; visual box size=0.01 0.01 0.01
- link joint5: geometry collision box size=0.01 0.01 0.01; visual box size=0.01 0.01 0.01
- link joint6: geometry collision box size=0.01 0.01 0.01; visual box size=0.01 0.01 0.01
- link joint6_flange: geometry collision box size=0.01 0.01 0.01; visual box size=0.01 0.01 0.01
Joints:
- removed joint apriltag_joint

File: mycobot_ros/mycobot_description/urdf/mycobot_pi/test_mycobot_urdf.urdf (robot description, URDF)
Before this commit: robot firefighter, 7 links, 6 joints
Links:
- link joint1: geometry collision mesh filename=package://mycobot_description/urdf/mycobot_pi/joint1_pi.dae; visual mesh filename=package://mycobot_description/urdf/mycobot_pi/joint1_pi.dae
- link joint2: geometry collision mesh filename=package://mycobot_description/urdf/mycobot_pi/joint2.dae; visual mesh filename=package://mycobot_description/urdf/mycobot_pi/joint2.dae
- link joint3: geometry collision mesh filename=package://mycobot_description/urdf/mycobot_pi/joint3.dae; visual mesh filename=package://mycobot_description/urdf/mycobot_pi/joint3.dae
- link joint4: geometry collision mesh filename=package://mycobot_description/urdf/mycobot_pi/joint4.dae; visual mesh filename=package://mycobot_description/urdf/mycobot_pi/joint4.dae
- link joint5: geometry collision mesh filename=package://mycobot_description/urdf/mycobot_pi/joint5.dae; visual mesh filename=package://mycobot_description/urdf/mycobot_pi/joint5.dae
- link joint6: geometry collision mesh filename=package://mycobot_description/urdf/mycobot_pi/joint6.dae; visual mesh filename=package://mycobot_description/urdf/mycobot_pi/joint6.dae
- link joint6_flange: geometry collision mesh filename=package://mycobot_description/urdf/mycobot_pi/joint7.dae; visual mesh filename=package://mycobot_description/urdf/mycobot_pi/joint7.dae
Joints:
- joint joint2_to_joint1: limit lower=-3.14 upper=3.14159 effort=1000.0 velocity=0 -> lower=-2.8624 upper=2.8624 effort=1000.0 velocity=0; origin xyz=0 0 0.13156 rpy=0 0 0 -> xyz=0 0 0.13956 rpy=0 0 0
- joint joint3_to_joint2: limit lower=-3.14 upper=3.14159 effort=1000.0 velocity=0 -> lower=-2.8624 upper=2.8624 effort=1000.0 velocity=0; origin xyz=0 0  0 rpy=0 1.5708 -1.5708 -> xyz=0 0 -0.001 rpy=0 1.5708 -1.5708
- joint joint4_to_joint3: limit lower=-3.14 upper=3.14159 effort=1000.0 velocity=0 -> lower=-2.8624 upper=2.8624 effort=1000.0 velocity=0
- joint joint5_to_joint4: limit lower=-3.14 upper=3.14159 effort=1000.0 velocity=0 -> lower=-2.8624 upper=2.8624 effort=1000.0 velocity=0
- joint joint6_to_joint5: limit lower=-3.14 upper=3.14159 effort=1000.0 velocity=0 -> lower=-2.8624 upper=2.8624 effort=1000.0 velocity=0
- joint joint6output_to_joint6: limit lower=-3.14 upper=3.14159 effort=1000.0 velocity=0 -> lower=-3.1241 upper=3.1241 effort=1000.0 velocity=0
